File: pat/ihc_mon.brd (EAGLE design)
At the start: 55.9 x 70.8 mm, 36 parts, among them IC1 PIC18F1220P, IC3 ADM3095EBRZ, X1 22-23-2021, X2 22-23-2021

Commit message: up
Connections:
- net N$19 renamed SIG4
- net N$22 renamed SIG5
Changed lines of the file:
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@@
 <?xml version="1.0" encoding="utf-8"?>
 <!DOCTYPE eagle SYSTEM "eagle.dtd">
-<eagle version="9.5.2">
+<eagle version="9.6.2">
 <drawing>
 <settings>
@@
 <wire x1="5.0292" y1="26.7462" x2="5.08" y2="26.67" width="0.254" layer="1"/>
 </signal>
-<signal name="N$19">
+<signal name="SIG4">
 <contactref element="IC1" pad="7"/>
 <contactref element="JP3" pad="4"/>
@@
 <wire x1="5.1435" y1="24.2316" x2="5.08" y2="24.13" width="0.254" layer="16"/>
 </signal>
-<signal name="N$22">
+<signal name="SIG5">
 <contactref element="IC1" pad="15"/>
 <contactref element="JP3" pad="5"/>
