File: pat/ihc_mon.sch (EAGLE design)
At the start: 36 parts, among them IC1 PIC18F1220P, IC3 ADM3095EBRZ, X1 22-23-2021, X2 22-23-2021

Commit message: up
Connections:
- net N$19 renamed SIG4
- net N$22 renamed SIG5
Changed lines of the file:
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@@
 <?xml version="1.0" encoding="utf-8"?>
 <!DOCTYPE eagle SYSTEM "eagle.dtd">
-<eagle version="9.5.2">
+<eagle version="9.6.2">
 <drawing>
 <settings>
@@
 </segment>
 </net>
-<net name="N$19" class="0">
+<net name="SIG4" class="0">
 <segment>
 <pinref part="IC1" gate="G$1" pin="RA3/AN3/VREF+"/>
@@
 </segment>
 </net>
-<net name="N$22" class="0">
+<net name="SIG5" class="0">
 <segment>
 <pinref part="IC1" gate="G$1" pin="RA6/CLKO/OSC2"/>
