File: host_board/mbmc_io.brd (EAGLE design)
At the start: 116.5 x 81.3 mm, 80 parts, among them IC1 ULN2803, IC2 DIP Socket, IC3 REF02 5 VOLTS, IC4 5 VOLTS, IC5 12 VOLTS, IC6 3.3 VOLTS, J1 1-1586043-4, J2 1586044-4

Commit message: up
Connections:
- net N$61 renamed 5VDC_REF
Changed lines of the file:
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@@
 <?xml version="1.0" encoding="utf-8"?>
 <!DOCTYPE eagle SYSTEM "eagle.dtd">
-<eagle version="9.5.2">
+<eagle version="9.6.2">
 <drawing>
 <settings>
@@
 <via x="54.7878" y="52.578" extent="1-16" drill="0.35"/>
 </signal>
-<signal name="N$61">
+<signal name="5VDC_REF">
 <contactref element="J1" pad="14"/>
 <contactref element="IC3" pad="6"/>
