File: host_board/mbmc_io.sch (EAGLE design)
At the start: 80 parts, among them IC1 ULN2803, IC2 DIP Socket, IC3 REF02 5 VOLTS, IC4 5 VOLTS, IC5 12 VOLTS, IC6 3.3 VOLTS, J1 1-1586043-4, J2 1586044-4

Commit message: up
Connections:
- net N$61 renamed 5VDC_REF
Changed lines of the file:
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@@
 <?xml version="1.0" encoding="utf-8"?>
 <!DOCTYPE eagle SYSTEM "eagle.dtd">
-<eagle version="9.5.2">
+<eagle version="9.6.2">
 <drawing>
 <settings>
@@
 </instance>
 <instance part="REFVDD" gate="G$1" x="-45.72" y="17.78" smashed="yes">
-<attribute name="NAME" x="-46.99" y="19.05" size="1.778" layer="95"/>
+<attribute name="NAME" x="-46.99" y="21.59" size="1.778" layer="95"/>
 <attribute name="TP_SIGNAL_NAME" x="-44.45" y="16.51" size="1.778" layer="97"/>
 </instance>
@@
 </instance>
 <instance part="REF24V" gate="G$1" x="-71.12" y="17.78" smashed="yes">
-<attribute name="NAME" x="-72.39" y="19.05" size="1.778" layer="95"/>
+<attribute name="NAME" x="-74.93" y="21.59" size="1.778" layer="95"/>
 <attribute name="TP_SIGNAL_NAME" x="-69.85" y="16.51" size="1.778" layer="97"/>
 </instance>
@@
 </segment>
 </net>
-<net name="N$61" class="0">
+<net name="5VDC_REF" class="0">
 <segment>
 <pinref part="J1" gate="G$1" pin="14"/>
@@
 <pinref part="VREF5VREF" gate="G$1" pin="TP"/>
 <junction x="-30.48" y="-43.18"/>
-</segment>
-</net>
+<label x="-45.72" y="96.52" size="1.778" layer="95"/>
+<label x="-27.94" y="-45.72" size="1.778" layer="95"/>
+<label x="-17.78" y="5.08" size="1.778" layer="95"/>
+</segment>
+</net>
