File: host_board/mbmc_single_board.brd (EAGLE design)
At the start: 116.5 x 81.3 mm, 118 parts, among them IC1 ULN2803, IC15 PIC18F57K42-E_PT, IC16 REF3440IDBVR, IC17 MAX232, IC2 DIP Socket, IC3 REF02 5 VOLTS, IC4 5 VOLTS, IC5 12 VOLTS, IC6 3.3 VOLTS, J1 1-1586043-4, J2 1586044-4, Q3 ASF1, X15 RX-2, X16 TX-2, X17 RESETJMP

Commit message: up
Connections:
- net N$234 renamed CLK16MHZCPU
- net N$235 renamed VREF4.1
- net N$243 renamed TX2
- net N$244 renamed RX1
- net N$252 renamed DLED
- net N$61 renamed VREF5V
- net N$89 renamed RX2
- net N$90 renamed TX1
Changed lines of the file:
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@@
 <?xml version="1.0" encoding="utf-8"?>
 <!DOCTYPE eagle SYSTEM "eagle.dtd">
-<eagle version="9.5.2">
+<eagle version="9.6.2">
 <drawing>
 <settings>
@@
 <via x="81.8388" y="44.577" extent="1-16" drill="0.35"/>
 </signal>
-<signal name="N$61">
+<signal name="VREF5V">
 <contactref element="J1" pad="14"/>
 <contactref element="IC3" pad="6"/>
@@
 <via x="48.768" y="13.0302" extent="1-16" drill="0.35"/>
 </signal>
-<signal name="N$234">
+<signal name="CLK16MHZCPU">
 <contactref element="Q3" pad="3"/>
 <contactref element="IC15" pad="32"/>
@@
 <via x="67.437" y="25.2222" extent="1-16" drill="0.35"/>
 </signal>
-<signal name="N$235">
+<signal name="VREF4.1">
 <contactref element="C60" pad="1"/>
 <contactref element="C57" pad="1"/>
@@
 <wire x1="22.86" y1="11.1252" x2="22.86" y2="11.11" width="0.1524" layer="1"/>
 </signal>
-<signal name="N$243">
+<signal name="TX2">
 <contactref element="IC17" pad="7"/>
 <contactref element="RS-232-3" pad="2"/>
@@
 <wire x1="24.1554" y1="3.81" x2="24.13" y2="3.81" width="0.1524" layer="1"/>
 </signal>
-<signal name="N$244">
+<signal name="RX1">
 <contactref element="IC17" pad="13"/>
 <contactref element="RS232-3" pad="3"/>
@@
 <via x="4.2672" y="47.7774" extent="1-16" drill="0.35"/>
 </signal>
-<signal name="N$252">
+<signal name="DLED">
 <contactref element="SV8" pad="4"/>
 <contactref element="IC15" pad="29"/>
@@
 <wire x1="55.8546" y1="2.5908" x2="55.88" y2="2.54" width="0.1524" layer="1"/>
 </signal>
-<signal name="N$89">
+<signal name="RX2">
 <contactref element="RS-232-3" pad="3"/>
 <contactref element="IC17" pad="8"/>
@@
 <wire x1="48.2346" y1="8.8392" x2="48.26" y2="8.89" width="0.1524" layer="16"/>
 </signal>
-<signal name="N$90">
+<signal name="TX1">
 <contactref element="RS232-3" pad="2"/>
 <contactref element="IC17" pad="14"/>

Commit message: up
Connections:
- net N$279 renamed EXT_INT1
- net N$290 renamed EXT_INT0
Changed lines of the file:
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@@
 <via x="78.0288" y="13.335" extent="1-16" drill="0.35"/>
 </signal>
-<signal name="N$279">
+<signal name="EXT_INT1">
 <contactref element="IC15" pad="9"/>
 <contactref element="U$1" pad="CH_L"/>
@@
 <via x="20.1168" y="22.6314" extent="1-16" drill="0.35"/>
 </signal>
-<signal name="N$290">
+<signal name="EXT_INT0">
 <contactref element="IC15" pad="8"/>
 <contactref element="C67" pad="1"/>

Commit message: up
Connections:
- net N$10 renamed ANB3_IN
- net N$21 renamed ULN2803_24VDC
- net N$24 renamed ANA1_IN
- net N$262 renamed ANA5
- net N$263 renamed ANA4
- net N$264 renamed ANA2
- net N$265 renamed ANA1
- net N$266 renamed ANA0
- net N$267 renamed ANA6
- net N$268 renamed IO_RF1
- net N$270 renamed SW0
- net N$271 renamed CALIB_B
- net N$272 renamed RELAYL1
- net N$273 renamed RELAYL2
- net N$274 renamed AC_CHARGER
- net N$275 renamed OUTP_3
- net N$276 renamed SELECT_B
- net N$277 renamed ENTER_B
- net N$278 renamed PWM8
- net N$280 renamed ANB2
- net N$281 renamed ANB4
- net N$282 renamed ANB5
- net N$283 renamed I5_ULN2803
- net N$284 renamed MAX_EN1
- net N$289 renamed ANB3
- net N$37 renamed DIP_P5
- net N$38 renamed DIP_P6
- net N$39 renamed DAQ_CS0
- net N$68 renamed ANA4_IN
- net N$69 renamed ANB4_IN
- net N$70 renamed ANA2_IN
- net N$71 renamed ANB5_IN
- net N$72 renamed ANA5_IN
- net N$73 renamed ANA6_IN
- net N$74 renamed ANA0_IN
- net N$8 renamed ANB2_IN
- net N$81 renamed DEBUG8_LED
- net N$84 renamed SL3_PIN3
Routing:
- net VSS: track 658.2 -> 655.5 mm

Commit message: up
Connections:
- net ANA0 renamed C_BATT
- net ANA0_IN renamed ANA0_IN_C_BAT
- net ANA1 renamed C_PV
- net ANA1_IN renamed ANA1_IN_C-PV
- net ANA2 renamed V_CC
- net ANA2_IN renamed ANA2_IN_V_CC
- net ANA4 renamed V_BAT
- net ANA4_IN renamed ANA4_IN_V_BAT
- net ANA5 renamed V_PV
- net ANA5_IN renamed ANA5_IN_V_PV
- net ANA6 renamed V_CMODE
- net ANA6_IN renamed ANA6_IN_V_CMODE
- net ANB2 renamed V_BBAT
- net ANB2_IN renamed ANB2_IN_V_BBAT
- net ANB3 renamed C_MPPT
- net ANB3_IN renamed ANB3_IN_C_MPPT
- net ANB4 renamed V_INVER
- net ANB4_IN renamed ANB4_IN_V_INVERTER
- net ANB5 renamed V_LIGHT_SEN
- net ANB5_IN renamed ANB5_IN_V_L_SENSOR
Routing:
- net VSS: track 655.5 -> 658.4 mm
Other:
- board text added: "FGB@NSASPOOK 2.0"
- board text removed: "FGB@MCHP 2.0"
Changed lines of the file:
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@@
 <hole x="3.81" y="77.47" drill="2.5"/>
 <text x="2.54" y="33.02" size="1.778" layer="1" font="vector" ratio="15" rot="R90">MBMC CPU/IO BOARD</text>
-<text x="2.54" y="12.7" size="1.778" layer="1" font="vector" ratio="15" rot="R90">FGB@MCHP 2.0</text>
+<text x="2.54" y="7.62" size="1.778" layer="1" font="vector" ratio="15" rot="R90">FGB@NSASPOOK 2.0</text>
 <text x="90.17" y="38.1" size="1.778" layer="1" font="vector" ratio="15" rot="R90">POWER</text>
 <text x="94.107" y="-6.35" size="0.0508" layer="200" font="vector" rot="R90">/fred/Downloads/mchp.bmp</text>
@@
 <wire x1="45.72" y1="35.5854" x2="45.72" y2="35.56" width="0.1524" layer="1"/>
 </signal>
-<signal name="ANB2_IN">
+<signal name="ANB2_IN_V_BBAT">
 <contactref element="R18" pad="2"/>
 <contactref element="J1" pad="7"/>
@@
 <wire x1="111.5568" y1="7.5438" x2="107.2134" y2="3.2004" width="0.3" layer="1"/>
 <wire x1="111.5568" y1="10.8204" x2="111.5568" y2="7.5438" width="0.3" layer="1"/>
-<wire x1="110.5662" y1="11.811" x2="111.5568" y2="10.8204" width="0.3" layer="1"/>
+<wire x1="110.49" y1="11.8872" x2="111.5568" y2="10.8204" width="0.3" layer="1"/>
 <wire x1="103.0224" y1="5.1054" x2="102.87" y2="5.08" width="0.3" layer="1"/>
 <wire x1="80.01" y1="38.1" x2="80.01" y2="35.56" width="0.3" layer="16"/>
@@
 <wire x1="110.5662" y1="19.6596" x2="110.49" y2="19.53" width="0.3" layer="1"/>
 <wire x1="110.5662" y1="27.051" x2="110.49" y2="27.15" width="0.3" layer="1"/>
-<wire x1="110.49" y1="34.7472" x2="110.49" y2="34.77" width="0" layer="19" extent="1-1"/>
-<wire x1="110.49" y1="27.15" x2="110.49" y2="29.337" width="0" layer="19" extent="1-1"/>
-<wire x1="110.5662" y1="11.811" x2="110.49" y2="11.91" width="0" layer="19" extent="1-1"/>
-<wire x1="110.3376" y1="27.1272" x2="110.49" y2="27.15" width="0" layer="19" extent="1-1"/>
-<wire x1="93.98" y1="16.99" x2="93.9546" y2="16.9926" width="0" layer="19" extent="1-1"/>
-<wire x1="74.93" y1="6.35" x2="75.057" y2="6.4008" width="0" layer="19" extent="1-1"/>
-<wire x1="74.9046" y1="6.3246" x2="74.93" y2="6.35" width="0" layer="19" extent="1-1"/>
+<wire x1="110.49" y1="34.8234" x2="110.49" y2="34.77" width="0.3" layer="1"/>
+<wire x1="110.49" y1="34.77" x2="110.49" y2="34.7472" width="0.3" layer="1"/>
+<wire x1="110.49" y1="27.15" x2="110.49" y2="29.337" width="0.3" layer="1"/>
+<wire x1="110.49" y1="11.8872" x2="110.49" y2="11.91" width="0.3" layer="1"/>
+<wire x1="74.9808" y1="6.4008" x2="74.93" y2="6.35" width="0.3" layer="1"/>
+<wire x1="74.93" y1="6.35" x2="74.9046" y2="6.3246" width="0.3" layer="1"/>
+<wire x1="74.9808" y1="6.3246" x2="74.93" y2="6.35" width="0.3" layer="1"/>
+<wire x1="74.9808" y1="6.3246" x2="75.057" y2="6.4008" width="0.3" layer="1"/>
+<wire x1="93.9546" y1="16.9926" x2="93.98" y2="16.99" width="0.3" layer="1"/>
+<wire x1="110.4138" y1="27.1272" x2="110.49" y2="27.15" width="0.3" layer="1"/>
+<wire x1="110.4138" y1="27.1272" x2="110.3376" y2="27.1272" width="0.3" layer="1"/>
 </signal>
-<signal name="ANA1_IN">
+<signal name="ANA1_IN_C-PV">
 <contactref element="J1" pad="2"/>
 <contactref element="R14" pad="1"/>
@@
 <wire x1="69.6468" y1="61.7982" x2="69.59" y2="61.81" width="0.1524" layer="16"/>
 </signal>
-<signal name="ANA2_IN">
+<signal name="ANA2_IN_V_CC">
 <contactref element="J1" pad="3"/>
 <contactref element="R15" pad="1"/>
@@
 <wire x1="48.6918" y1="67.2846" x2="48.64" y2="67.31" width="0.1524" layer="1"/>
 </signal>
-<signal name="ANA4_IN">
+<signal name="ANA4_IN_V_BAT">
 <contactref element="R16" pad="1"/>
 <contactref element="J1" pad="4"/>
@@
 <via x="30.3276" y="45.6438" extent="1-16" drill="0.35"/>
 </signal>
-<signal name="ANB4_IN">
+<signal name="ANB4_IN_V_INVERTER">
 <contactref element="R11" pad="1"/>
 <contactref element="J1" pad="9"/>
@@
 <via x="20.2692" y="74.1426" extent="1-16" drill="0.35"/>
 </signal>
-<signal name="ANB5_IN">
+<signal name="ANB5_IN_V_L_SENSOR">
 <contactref element="J1" pad="10"/>
 <contactref element="R20" pad="2"/>
@@
 <via x="43.8912" y="40.9956" extent="1-16" drill="0.35"/>
 </signal>
-<signal name="ANB3_IN">
+<signal name="ANB3_IN_C_MPPT">
 <contactref element="J1" pad="8"/>
 <contactref element="R19" pad="2"/>
@@
 <wire x1="56.9976" y1="61.7982" x2="57.02" y2="61.81" width="0.1524" layer="1"/>
 </signal>
-<signal name="ANA5_IN">
+<signal name="ANA5_IN_V_PV">
 <contactref element="R12" pad="1"/>
 <contactref element="J1" pad="5"/>
@@
 <via x="30.0228" y="60.4266" extent="1-16" drill="0.35"/>
 </signal>
-<signal name="ANA6_IN">
+<signal name="ANA6_IN_V_CMODE">
 <contactref element="R17" pad="1"/>
 <contactref element="J1" pad="6"/>
@@
 <via x="41.8338" y="51.1302" extent="1-16" drill="0.35"/>
 </signal>
-<signal name="ANA0_IN">
+<signal name="ANA0_IN_C_BAT">
 <contactref element="J1" pad="1"/>
 <contactref element="R13" pad="1"/>
@@
 <via x="72.4662" y="55.3212" extent="1-16" drill="0.35"/>
 </signal>
-<signal name="ANA5">
+<signal name="V_PV">
 <contactref element="IC15" pad="26"/>
 <contactref element="R5" pad="2"/>
@@
 <via x="39.7764" y="27.9654" extent="1-16" drill="0.35"/>
 </signal>
-<signal name="ANA4">
+<signal name="V_BAT">
 <contactref element="IC15" pad="25"/>
 <contactref element="R4" pad="2"/>
@@
 <via x="30.9372" y="34.5186" extent="1-16" drill="0.35"/>
 </signal>
-<signal name="ANA2">
+<signal name="V_CC">
 <contactref element="IC15" pad="23"/>
 <contactref element="R3" pad="2"/>
@@
 <via x="25.3746" y="27.1272" extent="1-16" drill="0.35"/>
 </signal>
-<signal name="ANA1">
+<signal name="C_PV">
 <contactref element="IC15" pad="22"/>
 <contactref element="R2" pad="2"/>
@@
 <via x="38.2524" y="26.9748" extent="1-16" drill="0.35"/>
 </signal>
-<signal name="ANA0">
+<signal name="C_BATT">
 <contactref element="IC15" pad="21"/>
 <contactref element="R1" pad="2"/>
@@
 <via x="61.5696" y="29.718" extent="1-16" drill="0.35"/>
 </signal>
-<signal name="ANA6">
+<signal name="V_CMODE">
 <contactref element="IC15" pad="33"/>
 <contactref element="R6" pad="2"/>
@@
 <via x="98.4504" y="23.0124" extent="1-16" drill="0.35"/>
 </signal>
-<signal name="ANB2">
+<signal name="V_BBAT">
 <contactref element="IC15" pad="10"/>
 <contactref element="R7" pad="2"/>
@@
 <via x="34.29" y="31.0896" extent="1-16" drill="0.35"/>
 </signal>
-<signal name="ANB4">
+<signal name="V_INVER">
 <contactref element="IC15" pad="16"/>
 <contactref element="R9" pad="2"/>
@@
 <via x="14.478" y="18.8214" extent="1-16" drill="0.35"/>
 </signal>
-<signal name="ANB5">
+<signal name="V_LIGHT_SEN">
 <contactref element="IC15" pad="17"/>
 <contactref element="R10" pad="2"/>
@@
 <via x="24.0792" y="40.767" extent="1-16" drill="0.35"/>
 </signal>
-<signal name="ANB3">
+<signal name="C_MPPT">
 <contactref element="IC15" pad="11"/>
 <contactref element="R8" pad="2"/>

Commit message: checkpoint
Connections:
- net N$49 renamed CAL_SW
Changed lines of the file:
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@@
 <wire x1="87.63" y1="5.1054" x2="87.63" y2="5.08" width="0.1524" layer="1"/>
 </signal>
-<signal name="N$49">
+<signal name="CAL_SW">
 <contactref element="INP" pad="4"/>
 <contactref element="U$1" pad="IN5"/>
