File: host_board/mbmc_single_board.sch (EAGLE design)
At the start: 118 parts, among them IC1 ULN2803, IC15 PIC18F57K42-E_PT, IC16 REF3440IDBVR, IC17 MAX232, IC2 DIP Socket, IC3 REF02 5 VOLTS, IC4 5 VOLTS, IC5 12 VOLTS, IC6 3.3 VOLTS, J1 1-1586043-4, J2 1586044-4, Q3 ASF1, X15 RX-2, X16 TX-2, X17 RESETJMP

Commit message: up
Connections:
- net N$234 renamed CLK16MHZCPU
- net N$235 renamed VREF4.1
- net N$243 renamed TX2
- net N$244 renamed RX1
- net N$252 renamed DLED
- net N$61 renamed VREF5V
- net N$89 renamed RX2
- net N$90 renamed TX1
Changed lines of the file:
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@@
 <?xml version="1.0" encoding="utf-8"?>
 <!DOCTYPE eagle SYSTEM "eagle.dtd">
-<eagle version="9.5.2">
+<eagle version="9.6.2">
 <drawing>
 <settings>
@@
 <pinref part="VSS35" gate="G$1" pin="VSS"/>
 <wire x1="-33.02" y1="-71.12" x2="-33.02" y2="-76.2" width="0.1524" layer="91"/>
+<junction x="-33.02" y="-76.2"/>
+<junction x="-33.02" y="-71.12"/>
 </segment>
 <segment>
@@
 <wire x1="-7.62" y1="-180.34" x2="2.54" y2="-180.34" width="0.1524" layer="91"/>
 <junction x="-7.62" y="-180.34"/>
+<junction x="2.54" y="-180.34"/>
 </segment>
 <segment>
@@
 <wire x1="-7.62" y1="-203.2" x2="2.54" y2="-203.2" width="0.1524" layer="91"/>
 <junction x="-7.62" y="-203.2"/>
+<junction x="2.54" y="-203.2"/>
 </segment>
 <segment>
@@
 <wire x1="-71.12" y1="-63.5" x2="-63.5" y2="-63.5" width="0.1524" layer="91"/>
 <junction x="-71.12" y="-63.5"/>
+<junction x="-63.5" y="-63.5"/>
 </segment>
 <segment>
@@
 <pinref part="+3V4" gate="G$1" pin="+3V3"/>
 <wire x1="-33.02" y1="-86.36" x2="-33.02" y2="-78.74" width="0.1524" layer="91"/>
+<junction x="-33.02" y="-78.74"/>
+<junction x="-33.02" y="-86.36"/>
 </segment>
 </net>
-<net name="N$61" class="0">
+<net name="VREF5V" class="0">
 <segment>
 <pinref part="J1" gate="G$1" pin="14"/>
@@
 <pinref part="VREF5VREF" gate="G$1" pin="TP"/>
 <junction x="-30.48" y="-43.18"/>
+<label x="-38.1" y="96.52" size="1.778" layer="95"/>
 </segment>
 </net>
@@
 </segment>
 </net>
-<net name="N$234" class="0">
+<net name="CLK16MHZCPU" class="0">
 <segment>
 <pinref part="IC15" gate="G$1" pin="RA7"/>
@@
 <label x="147.32" y="-200.66" size="1.778" layer="95"/>
 <junction x="144.78" y="-200.66"/>
+<label x="149.86" y="-228.6" size="1.778" layer="95"/>
 </segment>
 </net>
-<net name="N$235" class="0">
+<net name="VREF4.1" class="0">
 <segment>
 <pinref part="IC16" gate="G$1" pin="5"/>
@@
 <label x="147.32" y="-190.5" size="1.778" layer="95"/>
 <junction x="144.78" y="-190.5"/>
+<label x="165.1" y="-246.38" size="1.778" layer="95"/>
 </segment>
 <segment>
@@
 <label x="-2.54" y="68.58" size="1.778" layer="95"/>
 <junction x="17.78" y="68.58"/>
+<label x="-2.54" y="93.98" size="1.778" layer="95"/>
 </segment>
 </net>
@@
 </segment>
 </net>
-<net name="N$243" class="0">
+<net name="TX2" class="0">
 <segment>
 <pinref part="IC17" gate="G$1" pin="T2OUT"/>
@@
 <wire x1="-2.54" y1="-200.66" x2="-2.54" y2="-210.82" width="0.1524" layer="91"/>
 <junction x="-7.62" y="-200.66"/>
+<label x="0" y="-213.36" size="1.778" layer="95"/>
 </segment>
 </net>
-<net name="N$244" class="0">
+<net name="RX1" class="0">
 <segment>
 <pinref part="IC17" gate="G$1" pin="R1IN"/>
@@
 <junction x="-7.62" y="-175.26"/>
 <junction x="53.34" y="-200.66"/>
+<label x="0" y="-175.26" size="1.778" layer="95"/>
 </segment>
 </net>
@@
 </segment>
 </net>
-<net name="N$252" class="0">
+<net name="DLED" class="0">
 <segment>
 <pinref part="SV8" gate="1" pin="4"/>
@@
 <junction x="190.5" y="-198.12"/>
 <junction x="190.5" y="-180.34"/>
+<label x="185.42" y="-200.66" size="1.778" layer="95"/>
 </segment>
 </net>
@@
 </segment>
 </net>
-<net name="N$89" class="0">
+<net name="RX2" class="0">
 <segment>
 <pinref part="RS-232-3" gate="G$1" pin="3"/>
@@
 <junction x="-7.62" y="-198.12"/>
 <junction x="53.34" y="-203.2"/>
+<label x="0" y="-198.12" size="1.778" layer="95"/>
 </segment>
 </net>
-<net name="N$90" class="0">
+<net name="TX1" class="0">
 <segment>
 <pinref part="RS232-3" gate="G$1" pin="2"/>
@@
 <junction x="-7.62" y="-177.8"/>
 <junction x="53.34" y="-195.58"/>
+<label x="0" y="-177.8" size="1.778" layer="95"/>
 </segment>
 </net>

Commit message: up
Connections:
- net N$279 renamed EXT_INT1
- net N$290 renamed EXT_INT0
Changed lines of the file:
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@@
 </segment>
 </net>
-<net name="N$279" class="0">
+<net name="EXT_INT1" class="0">
 <segment>
 <pinref part="IC15" gate="G$1" pin="RB1"/>
@@
 </segment>
 </net>
-<net name="N$290" class="0">
+<net name="EXT_INT0" class="0">
 <segment>
 <pinref part="C67" gate="G$1" pin="1"/>

Commit message: up
Connections:
- net N$10 renamed ANB3_IN
- net N$21 renamed ULN2803_24VDC
- net N$24 renamed ANA1_IN
- net N$262 renamed ANA5
- net N$263 renamed ANA4
- net N$264 renamed ANA2
- net N$265 renamed ANA1
- net N$266 renamed ANA0
- net N$267 renamed ANA6
- net N$268 renamed IO_RF1
- net N$270 renamed SW0
- net N$271 renamed CALIB_B
- net N$272 renamed RELAYL1
- net N$273 renamed RELAYL2
- net N$274 renamed AC_CHARGER
- net N$275 renamed OUTP_3
- net N$276 renamed SELECT_B
- net N$277 renamed ENTER_B
- net N$278 renamed PWM8
- net N$280 renamed ANB2
- net N$281 renamed ANB4
- net N$282 renamed ANB5
- net N$283 renamed I5_ULN2803
- net N$284 renamed MAX_EN1
- net N$289 renamed ANB3
- net N$37 renamed DIP_P5
- net N$38 renamed DIP_P6
- net N$39 renamed DAQ_CS0
- net N$68 renamed ANA4_IN
- net N$69 renamed ANB4_IN
- net N$70 renamed ANA2_IN
- net N$71 renamed ANB5_IN
- net N$72 renamed ANA5_IN
- net N$73 renamed ANA6_IN
- net N$74 renamed ANA0_IN
- net N$8 renamed ANB2_IN
- net N$81 renamed DEBUG8_LED
- net N$84 renamed SL3_PIN3

Commit message: up
Connections:
- net ANA0 renamed C_BATT
- net ANA0_IN renamed ANA0_IN_C_BAT
- net ANA1 renamed C_PV
- net ANA1_IN renamed ANA1_IN_C-PV
- net ANA2 renamed V_CC
- net ANA2_IN renamed ANA2_IN_V_CC
- net ANA4 renamed V_BAT
- net ANA4_IN renamed ANA4_IN_V_BAT
- net ANA5 renamed V_PV
- net ANA5_IN renamed ANA5_IN_V_PV
- net ANA6 renamed V_CMODE
- net ANA6_IN renamed ANA6_IN_V_CMODE
- net ANB2 renamed V_BBAT
- net ANB2_IN renamed ANB2_IN_V_BBAT
- net ANB3 renamed C_MPPT
- net ANB3_IN renamed ANB3_IN_C_MPPT
- net ANB4 renamed V_INVER
- net ANB4_IN renamed ANB4_IN_V_INVERTER
- net ANB5 renamed V_LIGHT_SEN
- net ANB5_IN renamed ANB5_IN_V_L_SENSOR
Changed lines of the file:
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@@
 </instance>
 <instance part="R18" gate="G$1" x="78.74" y="76.2" smashed="yes">
-<attribute name="NAME" x="74.93" y="77.6986" size="1.778" layer="95"/>
-<attribute name="VALUE" x="74.93" y="72.898" size="1.778" layer="96"/>
+<attribute name="NAME" x="82.55" y="75.1586" size="1.778" layer="95"/>
+<attribute name="VALUE" x="80.01" y="70.358" size="1.778" layer="96"/>
 </instance>
 <instance part="R19" gate="G$1" x="99.06" y="76.2" smashed="yes">
 <attribute name="NAME" x="95.25" y="77.6986" size="1.778" layer="95"/>
-<attribute name="VALUE" x="95.25" y="72.898" size="1.778" layer="96"/>
+<attribute name="VALUE" x="102.87" y="77.978" size="1.778" layer="96"/>
 </instance>
 <instance part="R20" gate="G$1" x="68.58" y="60.96" smashed="yes">
@@
 <instance part="R24" gate="G$1" x="93.98" y="81.28" smashed="yes">
 <attribute name="NAME" x="90.17" y="82.7786" size="1.778" layer="95"/>
-<attribute name="VALUE" x="90.17" y="77.978" size="1.778" layer="96"/>
+<attribute name="VALUE" x="87.63" y="77.978" size="1.778" layer="96"/>
 </instance>
 <instance part="R25" gate="G$1" x="45.72" y="63.5" smashed="yes">
@@
 </instance>
 <instance part="VSS6" gate="G$1" x="68.58" y="68.58" smashed="yes" rot="R180">
-<attribute name="VALUE" x="71.12" y="73.66" size="1.778" layer="96" rot="R270"/>
+<attribute name="VALUE" x="68.58" y="68.58" size="1.778" layer="96" rot="R270"/>
 </instance>
 <instance part="VSS7" gate="G$1" x="83.82" y="68.58" smashed="yes" rot="R180">
@@
 <pinref part="R1" gate="G$1" pin="E"/>
 <pinref part="R13" gate="G$1" pin="2"/>
+<junction x="43.18" y="93.98"/>
 </segment>
 </net>
@@
 </segment>
 </net>
-<net name="ANB2_IN" class="0">
+<net name="ANB2_IN_V_BBAT" class="0">
 <segment>
 <pinref part="R18" gate="G$1" pin="2"/>
@@
 <junction x="83.82" y="76.2"/>
 <label x="-45.72" y="73.66" size="1.778" layer="95"/>
+<label x="63.5" y="73.66" size="1.778" layer="95"/>
 </segment>
 </net>
@@
 </segment>
 </net>
-<net name="ANA1_IN" class="0">
+<net name="ANA1_IN_C-PV" class="0">
 <segment>
 <pinref part="J1" gate="G$1" pin="2"/>
@@
 <junction x="48.26" y="91.44"/>
 <label x="-45.72" y="60.96" size="1.778" layer="95"/>
+<label x="43.18" y="96.52" size="1.778" layer="95"/>
 </segment>
 </net>
@@
 </segment>
 </net>
-<net name="ANA2_IN" class="0">
+<net name="ANA2_IN_V_CC" class="0">
 <segment>
 <pinref part="J1" gate="G$1" pin="3"/>
@@
 <junction x="63.5" y="91.44"/>
 <label x="-45.72" y="63.5" size="1.778" layer="95"/>
+<label x="63.5" y="96.52" size="1.778" layer="95"/>
 </segment>
 </net>
-<net name="ANA4_IN" class="0">
+<net name="ANA4_IN_V_BAT" class="0">
 <segment>
 <pinref part="R16" gate="G$1" pin="1"/>
@@
 <junction x="78.74" y="91.44"/>
 <label x="-45.72" y="66.04" size="1.778" layer="95"/>
+<label x="83.82" y="96.52" size="1.778" layer="95"/>
 </segment>
 </net>
-<net name="ANB4_IN" class="0">
+<net name="ANB4_IN_V_INVERTER" class="0">
 <segment>
 <pinref part="R11" gate="G$1" pin="1"/>
@@
 <junction x="-48.26" y="78.74"/>
 <label x="-45.72" y="78.74" size="1.778" layer="95"/>
+<label x="27.94" y="45.72" size="1.778" layer="95"/>
 </segment>
 </net>
-<net name="ANB5_IN" class="0">
+<net name="ANB5_IN_V_L_SENSOR" class="0">
 <segment>
 <pinref part="J1" gate="G$1" pin="10"/>
@@
 <junction x="73.66" y="60.96"/>
 <label x="-45.72" y="81.28" size="1.778" layer="95"/>
+<label x="58.42" y="45.72" size="1.778" layer="95"/>
 </segment>
 </net>
@@
 </segment>
 </net>
-<net name="ANB3_IN" class="0">
+<net name="ANB3_IN_C_MPPT" class="0">
 <segment>
 <pinref part="J1" gate="G$1" pin="8"/>
@@
 <wire x1="104.14" y1="76.2" x2="101.6" y2="76.2" width="0.1524" layer="91"/>
 <label x="-45.72" y="76.2" size="1.778" layer="95"/>
+<label x="91.44" y="73.66" size="1.778" layer="95"/>
 </segment>
 </net>
-<net name="ANA5_IN" class="0">
+<net name="ANA5_IN_V_PV" class="0">
 <segment>
 <pinref part="R12" gate="G$1" pin="1"/>
@@
 <junction x="33.02" y="76.2"/>
 <label x="-45.72" y="68.58" size="1.778" layer="95"/>
+<label x="33.02" y="78.74" size="1.778" layer="95"/>
 </segment>
 </net>
-<net name="ANA6_IN" class="0">
+<net name="ANA6_IN_V_CMODE" class="0">
 <segment>
 <pinref part="R17" gate="G$1" pin="1"/>
@@
 <junction x="53.34" y="66.04"/>
 <label x="-45.72" y="71.12" size="1.778" layer="95"/>
+<label x="48.26" y="76.2" size="1.778" layer="95"/>
 </segment>
 </net>
-<net name="ANA0_IN" class="0">
+<net name="ANA0_IN_C_BAT" class="0">
 <segment>
 <wire x1="20.32" y1="101.6" x2="20.32" y2="93.98" width="0.1524" layer="91"/>
@@
 <junction x="33.02" y="93.98"/>
 <label x="-45.72" y="58.42" size="1.778" layer="95"/>
+<label x="20.32" y="96.52" size="1.778" layer="95"/>
 </segment>
 </net>
@@
 </segment>
 </net>
-<net name="ANA5" class="0">
+<net name="V_PV" class="0">
 <segment>
 <pinref part="IC15" gate="G$1" pin="RA5"/>
@@
 </segment>
 </net>
-<net name="ANA4" class="0">
+<net name="V_BAT" class="0">
 <segment>
 <pinref part="IC15" gate="G$1" pin="RA4"/>
@@
 </segment>
 </net>
-<net name="ANA2" class="0">
+<net name="V_CC" class="0">
 <segment>
 <pinref part="IC15" gate="G$1" pin="RA2"/>
@@
 </segment>
 </net>
-<net name="ANA1" class="0">
+<net name="C_PV" class="0">
 <segment>
 <pinref part="IC15" gate="G$1" pin="RA1"/>
@@
 </segment>
 </net>
-<net name="ANA0" class="0">
+<net name="C_BATT" class="0">
 <segment>
 <pinref part="IC15" gate="G$1" pin="RA0"/>
@@
 </segment>
 </net>
-<net name="ANA6" class="0">
+<net name="V_CMODE" class="0">
 <segment>
 <pinref part="IC15" gate="G$1" pin="RA6"/>
@@
 </segment>
 </net>
-<net name="ANB2" class="0">
+<net name="V_BBAT" class="0">
 <segment>
 <pinref part="IC15" gate="G$1" pin="RB2"/>
@@
 </segment>
 </net>
-<net name="ANB4" class="0">
+<net name="V_INVER" class="0">
 <segment>
 <pinref part="IC15" gate="G$1" pin="RB4"/>
@@
 </segment>
 </net>
-<net name="ANB5" class="0">
+<net name="V_LIGHT_SEN" class="0">
 <segment>
 <pinref part="IC15" gate="G$1" pin="RB5"/>
@@
 </segment>
 </net>
-<net name="ANB3" class="0">
+<net name="C_MPPT" class="0">
 <segment>
 <pinref part="IC15" gate="G$1" pin="RB3"/>

Commit message: checkpoint
Connections:
- net N$49 renamed CAL_SW
Changed lines of the file:
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@@
 </segment>
 </net>
-<net name="N$49" class="0">
+<net name="CAL_SW" class="0">
 <segment>
 <pinref part="INP" gate="-4" pin="S"/>
@@
 <junction x="119.38" y="2.54"/>
 <junction x="142.24" y="-27.94"/>
+<label x="134.62" y="-27.94" size="1.778" layer="95"/>
+<label x="96.52" y="2.54" size="1.778" layer="95"/>
 </segment>
 </net>
@@
 <label x="27.94" y="0" size="1.778" layer="95"/>
 <junction x="25.4" y="0"/>
-</segment>
-</net>
+<label x="134.62" y="-63.5" size="1.778" layer="95"/>
+<label x="198.12" y="-27.94" size="1.778" layer="95"/>
+</segment>
+</net>
