File: host_board/hall_sensor100a.brd (EAGLE design)
At the start: 60.6 x 57.1 mm, 29 parts, among them IC1 REF02HCSA, IC2 CSLT6B100, IC3 MAX5322EAI+, X1 22-23-2051

Commit message: up
Connections:
- net N$1 renamed 5VDC_REG
- net N$2 renamed SENSOR_OUT
Changed lines of the file:
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@@
 <via x="62.484" y="38.0238" extent="1-16" drill="0.35"/>
 </signal>
-<signal name="N$2">
+<signal name="SENSOR_OUT">
 <contactref element="IC2" pad="3"/>
 <contactref element="X1" pad="2"/>
@@
 <wire x1="27.9654" y1="39.3192" x2="27.94" y2="39.37" width="0.1524" layer="16"/>
 </signal>
-<signal name="N$1" class="1">
+<signal name="5VDC_REG" class="1">
 <contactref element="IC2" pad="1"/>
 <contactref element="IC1" pad="6"/>
