File: host_board/hall_sensor100a.sch (EAGLE design)
At the start: 29 parts, among them IC1 REF02HCSA, IC2 CSLT6B100, IC3 MAX5322EAI+, X1 22-23-2051

Commit message: up
Connections:
- net N$1 renamed 5VDC_REG
- net N$2 renamed SENSOR_OUT
Other:
- note added: "gnd/black/drain 1 sensor white 2 5vdc reg green 3 +12vdc red 4"
Changed lines of the file:
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@@
 <?xml version="1.0" encoding="utf-8"?>
 <!DOCTYPE eagle SYSTEM "eagle.dtd">
-<eagle version="9.5.2">
+<eagle version="9.6.2">
 <drawing>
 <settings>
@@
 <sheet>
 <plain>
+<text x="114.3" y="50.8" size="1.778" layer="91">gnd/black/drain           1
+sensor  white                2
+5vdc reg  green            3
++12vdc red                    4</text>
 </plain>
 <instances>
@@
 <junction x="93.98" y="50.8"/>
 <junction x="101.6" y="53.34"/>
+<label x="96.52" y="53.34" size="1.778" layer="95"/>
 </segment>
 <segment>
@@
 </segment>
 </net>
-<net name="N$2" class="0">
+<net name="SENSOR_OUT" class="0">
 <segment>
 <pinref part="IC2" gate="G$1" pin="OUTPUT"/>
@@
 <junction x="96.52" y="68.58"/>
 <junction x="119.38" y="68.58"/>
-</segment>
-</net>
-<net name="N$1" class="1">
+<label x="45.72" y="73.66" size="1.778" layer="95"/>
+</segment>
+</net>
+<net name="5VDC_REG" class="1">
 <segment>
 <pinref part="IC2" gate="G$1" pin="VS_(+)"/>
@@
 <junction x="119.38" y="73.66"/>
 <wire x1="119.38" y1="73.66" x2="121.92" y2="73.66" width="0.1524" layer="91"/>
+<label x="78.74" y="66.04" size="1.778" layer="95"/>
 </segment>
 </net>
@@
 </drawing>
 <compatibility>
+<note version="6.3" minversion="6.2.2" severity="warning">
+Since Version 6.2.2 text objects can contain more than one line,
+which will not be processed correctly with this version.
+</note>
 <note version="8.2" severity="warning">
 Since Version 8.2, EAGLE supports online libraries. The ids
